File: canSim.brd (EAGLE design)
At the start: 98.7 x 87.6 mm, 16 parts

Commit message: New revision with new OBD-2.  Auto PCB routing to still change.
Parts:
- U$9: value OBD_2FEMALE -> OBD_2FEMALEOBD2_FEMALE_PTH
- moved U$2 58.5 mm to (83.8, 31.8)
- moved U$3 58.5 mm to (25.4, 31.8)
- moved U$8 15.3 mm to (101.0, 64.8)
- moved H2 6.48 mm to (95.2, 3.81)
- moved H3 6.35 mm to (44.5, 3.81)
- moved U$11 5.21 mm to (64.5, 69.8)
- moved U$5 4.58 mm to (16.5, 67.3)
- moved U$1 3.81 mm to (26.7, 67.3)
- moved U$4 3.81 mm to (54.6, 31.8)
- moved H5 3.81 mm to (3.81, 14.0)
- moved U$6 3.81 mm to (2.54, 33.0)
- moved H1 3.81 mm to (95.2, 80.0)
- moved H4 3.81 mm to (3.81, 80.0)
- moved U$10 3.00 mm to (83.8, 3.00)
- moved U$7 3.00 mm to (54.6, 3.00)
Routing:
- net CAN2_P: track 75.3 -> 0.00 mm
- net CAN2_N: track 75.2 -> 0.00 mm
- net CAN3_N: track 55.2 -> 0.00 mm
- net CAN3_P: track 55.2 -> 0.00 mm
- net CAN1_P: track 29.2 -> 0.00 mm
- net CAN1_N: track 29.2 -> 0.00 mm
Other:
- board size 98.7 x 87.6 mm -> 98.7 x 83.8 mm

Commit message: board file
Routing:
- net +3V3: track 0.00 -> 190.9 mm, vias 0 -> 2
- net +5V: track 0.00 -> 167.7 mm
- net ENC_BTN: track 0.00 -> 126.2 mm
- net MISO_5: track 0.00 -> 125.8 mm, vias 0 -> 1
- net ENC_B: track 0.00 -> 98.8 mm, vias 0 -> 1
- net ENC_A: track 0.00 -> 89.5 mm, vias 0 -> 2
- net INT1_5: track 0.00 -> 87.5 mm, vias 0 -> 2
- net SD_CMD: track 0.00 -> 85.7 mm, vias 0 -> 1
- net SD_DAT2: track 0.00 -> 85.5 mm, vias 0 -> 1
- net SCK: track 0.00 -> 77.5 mm, vias 0 -> 1
- net CS1: track 0.00 -> 77.0 mm, vias 0 -> 1
- net SD_DAT0: track 0.00 -> 76.3 mm, vias 0 -> 1
- net CAN1_N: track 0.00 -> 75.2 mm
- net SDA: track 0.00 -> 73.5 mm, vias 0 -> 1
- net CS2: track 0.00 -> 72.8 mm, vias 0 -> 1
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
Commit message: Release candidate
Parts:
- added R1, R2: 10k, resistor:0207/2V
- added T1: 2N3904, transistor:TO92
- moved U$6 6.35 mm to (2.54, 26.7)
- moved H1 1.00 mm to (96.2, 80.0)
- moved H2 1.00 mm to (96.2, 3.81)
Connections:
- new net COLL: R2.1, T1.1, U$6.P$2
- new net N$2: R1.2, T1.2
- net +5V: now also R2.2
- net 12V_EN: now also R1.1; no longer U$6.P$2
- net GND: now also T1.3
Routing:
- net +5V: track 167.7 -> 229.9 mm, vias 0 -> 2
- net +3V3: track 190.9 -> 219.4 mm, vias 2 -> 0
- net MISO_5: track 125.8 -> 99.3 mm, vias 1 -> 4
- net SD_DAT2: track 85.5 -> 63.1 mm, vias 1 -> 0
- net CS1: track 77.0 -> 58.6 mm, vias 1 -> 2
- net SDA: track 73.5 -> 56.8 mm, vias 1 -> 0
- net COLL: track 0.00 -> 16.6 mm
- net SD_CD: track 67.6 -> 84.2 mm, vias 1 -> 2
- net 12V_EN: track 67.5 -> 51.0 mm, vias 0 -> 1
- net +12V: track 47.6 -> 62.1 mm
- net INT1_5: track 87.5 -> 74.0 mm, vias 2 -> 0
- net SD_DAT0: track 76.3 -> 63.0 mm, vias 1 -> 0
- net SD_CLK: track 66.5 -> 79.6 mm, vias 1 -> 0
- net SD_CMD: track 85.7 -> 74.0 mm, vias 1 -> 0
- net CS3: track 51.9 -> 41.8 mm, vias 2 -> 3
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- added copper zone on layer 1, net GND
Other:
- board size 98.7 x 83.8 mm -> 100 x 83.8 mm
- board text added: "(c)2020-2021 J. Bordens USE AT YOUR OWN RISK! THIS BOARD IS PROVIDED "AS IS", WITHOUT WARRANTY OF ANY KIND, EXPRESS OR IMPLIED. The copyright holder disclaims all liability for damages resulting from use of this board to the fullest extent possible."

Commit message: Minor tweaks - moved connector. Shifter hole size.
Moved connector down a little for better fit with the real connector.
Bigger holes for the 3.3v-5v level shifter so you can use real headers.
Parts:
- moved U$9 1.00 mm to (20.3, -1.00)
Routing:
- net +12V: track 62.1 -> 50.1 mm
- net CAN2_P: track 23.3 -> 24.5 mm
- net CAN2_N: track 23.5 -> 24.7 mm
- net CAN3_N: track 48.6 -> 49.6 mm
- net CAN1_N: track 68.2 -> 69.2 mm
- net CAN1_P: track 68.5 -> 69.5 mm
- net CAN3_P: track 49.5 -> 50.4 mm

Commit message: Swap interrupt and CS pins because some ESP32 pins are input-only.
Parts:
- moved H5 0.25 mm to (3.56, 14.0)
- moved H1 0.25 mm to (96.2, 80.3)
Connections:
- net CS2: now also U$1.D32; no longer U$1.D39
- net CS3: now also U$1.D33; no longer U$1.D34
- net INT2_3V3: now also U$1.D34; no longer U$1.D32
- net INT3_3V3: now also U$1.D39; no longer U$1.D33
Routing:
- net INT3_3V3: track 22.4 -> 32.8 mm
- net CS2: track 75.5 -> 67.9 mm
- net INT2_3V3: track 20.7 -> 25.8 mm
- net CS3: track 41.8 -> 45.0 mm
Changed lines of the file:
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@@
 <setting verticaltext="up"/>
 </settings>
-<grid distance="10" unitdist="mil" unit="mil" style="lines" multiple="1" display="yes" altdistance="5" altunitdist="mil" altunit="mil"/>
+<grid distance="10" unitdist="mil" unit="mm" style="lines" multiple="1" display="yes" altdistance="5" altunitdist="mil" altunit="mil"/>
 <layers>
 <layer number="1" name="Top" color="4" fill="1" visible="yes" active="yes"/>
@@
 <element name="U$7" library="cheap_oled" package="128X64_SQUARE_VERT" value="128X64_SQUARE" x="54.61" y="3" smashed="yes"/>
 <element name="U$10" library="cheap_encoder" package="CHEAP_ENCODER_VERT" value="ROTARY_ENC" x="83.82" y="3" smashed="yes"/>
-<element name="H1" library="holes" library_urn="urn:adsk.eagle:library:237" package="2,8" package3d_urn="urn:adsk.eagle:package:14271/1" value="MOUNT-HOLE2.8" x="96.25" y="80.01" smashed="yes">
-<attribute name="POPULARITY" value="15" x="96.25" y="80.01" size="1.778" layer="27" display="off"/>
+<element name="H1" library="holes" library_urn="urn:adsk.eagle:library:237" package="2,8" package3d_urn="urn:adsk.eagle:package:14271/1" value="MOUNT-HOLE2.8" x="96.25" y="80.264" smashed="yes">
+<attribute name="POPULARITY" value="15" x="96.25" y="80.264" size="1.778" layer="27" display="off"/>
 </element>
 <element name="H2" library="holes" library_urn="urn:adsk.eagle:library:237" package="2,8" package3d_urn="urn:adsk.eagle:package:14271/1" value="MOUNT-HOLE2.8" x="96.25" y="3.81" smashed="yes">
@@
 <attribute name="POPULARITY" value="15" x="3.81" y="80.01" size="1.778" layer="27" display="off"/>
 </element>
-<element name="H5" library="holes" library_urn="urn:adsk.eagle:library:237" package="2,8" package3d_urn="urn:adsk.eagle:package:14271/1" value="MOUNT-HOLE2.8" x="3.81" y="13.97" smashed="yes">
-<attribute name="POPULARITY" value="15" x="3.81" y="13.97" size="1.778" layer="27" display="off"/>
+<element name="H5" library="holes" library_urn="urn:adsk.eagle:library:237" package="2,8" package3d_urn="urn:adsk.eagle:package:14271/1" value="MOUNT-HOLE2.8" x="3.556" y="13.97" smashed="yes">
+<attribute name="POPULARITY" value="15" x="3.556" y="13.97" size="1.778" layer="27" display="off"/>
 </element>
 <element name="U$11" library="cheap_power_jack" package="CHEAP_POWER_JACK" value="CHEAP_POWER_JACK" x="64.516" y="69.85" smashed="yes"/>
@@
 </signal>
 <signal name="CS2">
-<contactref element="U$1" pad="D39"/>
 <contactref element="U$3" pad="P$5"/>
 <wire x1="7.7089" y1="73.5711" x2="7.62" y2="73.66" width="0.4064" layer="16"/>
@@
 <via x="19.05" y="74.93" extent="1-16" drill="0.35"/>
 <wire x1="19.05" y1="74.93" x2="19.1361" y2="75.0161" width="0.4064" layer="1"/>
-<wire x1="19.1361" y1="75.0161" x2="40.64" y2="75.0161" width="0.4064" layer="1"/>
-<via x="40.64" y="75.0161" extent="1-16" drill="0.35"/>
-<wire x1="40.64" y1="75.0161" x2="40.63" y2="75.0261" width="0.4064" layer="16"/>
-<wire x1="40.63" y1="75.0261" x2="40.63" y2="80.445" width="0.4064" layer="16"/>
+<wire x1="19.1361" y1="75.0161" x2="33.02" y2="75.0161" width="0.4064" layer="1"/>
+<via x="33.02" y="75.0161" extent="1-16" drill="0.35"/>
+<contactref element="U$1" pad="D32"/>
+<wire x1="33.02" y1="75.0161" x2="33.01" y2="75.0261" width="0.4064" layer="16"/>
+<wire x1="33.01" y1="75.0261" x2="33.01" y2="80.445" width="0.4064" layer="16"/>
 </signal>
 <signal name="CS3">
-<contactref element="U$1" pad="D34"/>
 <contactref element="U$4" pad="P$5"/>
-<wire x1="38.09" y1="80.445" x2="38.09" y2="73.67" width="0.4064" layer="16"/>
-<wire x1="38.09" y1="73.67" x2="38.1" y2="73.66" width="0.4064" layer="16"/>
-<via x="38.1" y="73.66" extent="1-16" drill="0.35"/>
-<wire x1="38.1" y1="73.66" x2="38.1" y2="63.628575" width="0.4064" layer="1"/>
-<wire x1="38.1" y1="63.628575" x2="38.110159375" y2="63.618415625" width="0.4064" layer="1"/>
+<via x="33.02" y="71.628" extent="1-16" drill="0.35"/>
+<wire x1="33.02" y1="71.628" x2="33.02" y2="68.708575" width="0.4064" layer="1"/>
+<wire x1="33.02" y1="68.708575" x2="38.110159375" y2="63.618415625" width="0.4064" layer="1"/>
 <via x="38.110159375" y="63.618415625" extent="1-16" drill="0.35"/>
 <wire x1="52.07" y1="54.61" x2="49.926696875" y2="56.753303125" width="0.4064" layer="16"/>
@@
 <via x="52.07" y="54.61" extent="1-16" drill="0.35"/>
 <wire x1="52.07" y1="54.61" x2="52.07" y2="50.363" width="0.4064" layer="1"/>
+<contactref element="U$1" pad="D33"/>
+<wire x1="33.02" y1="71.628" x2="31.75" y2="72.898" width="0.4064" layer="16"/>
+<wire x1="31.75" y1="79.165" x2="30.47" y2="80.445" width="0.4064" layer="16"/>
+<wire x1="31.75" y1="72.898" x2="31.75" y2="79.165" width="0.4064" layer="16"/>
 </signal>
 <signal name="+3V3" class="1">
@@
 </signal>
 <signal name="INT2_3V3">
-<contactref element="U$1" pad="D32"/>
 <contactref element="U$5" pad="P$11"/>
 <wire x1="21.59" y1="72.39" x2="22.86" y2="71.12" width="0.4064" layer="16"/>
@@
 <via x="27.94" y="72.3039" extent="1-16" drill="0.35"/>
 <wire x1="27.94" y1="72.3039" x2="27.8991" y2="72.898" width="0.4064" layer="1"/>
-<wire x1="27.8991" y1="72.898" x2="32.893" y2="72.898" width="0.4064" layer="1"/>
-<wire x1="32.893" y1="72.898" x2="33.02" y2="72.8571" width="0.4064" layer="1"/>
-<via x="33.02" y="72.8571" extent="1-16" drill="0.35"/>
-<wire x1="33.02" y1="72.8571" x2="33.01" y2="72.8671" width="0.4064" layer="16"/>
-<wire x1="33.01" y1="72.8671" x2="33.01" y2="80.445" width="0.4064" layer="16"/>
+<wire x1="27.8991" y1="72.898" x2="37.973" y2="72.898" width="0.4064" layer="1"/>
+<wire x1="37.973" y1="72.898" x2="38.1" y2="72.8571" width="0.4064" layer="1"/>
+<via x="38.1" y="72.8571" extent="1-16" drill="0.35"/>
 <wire x1="22.86" y1="71.12" x2="26.543" y2="71.12" width="0.4064" layer="16"/>
 <wire x1="26.543" y1="71.12" x2="27.7269" y2="72.3039" width="0.4064" layer="16"/>
+<contactref element="U$1" pad="D34"/>
+<wire x1="38.1" y1="72.8571" x2="38.09" y2="72.8671" width="0.4064" layer="16"/>
+<wire x1="38.09" y1="72.8671" x2="38.09" y2="80.445" width="0.4064" layer="16"/>
 </signal>
 <signal name="INT3_3V3">
-<contactref element="U$1" pad="D33"/>
 <contactref element="U$5" pad="P$8"/>
-<via x="30.48" y="75.946" extent="1-16" drill="0.35"/>
+<via x="40.64" y="75.692" extent="1-16" drill="0.35"/>
 <wire x1="13.97" y1="72.39" x2="14.89910625" y2="72.39" width="0.4064" layer="1"/>
-<wire x1="29.9664" y1="75.6638" x2="30.48" y2="75.946" width="0.4064" layer="1"/>
+<wire x1="40.588675" y1="75.6638" x2="40.64" y2="75.692" width="0.4064" layer="1"/>
 <wire x1="14.89910625" y1="72.39" x2="18.17290625" y2="75.6638" width="0.4064" layer="1"/>
-<wire x1="18.17290625" y1="75.6638" x2="29.9664" y2="75.6638" width="0.4064" layer="1"/>
-<wire x1="30.48" y1="75.946" x2="30.47" y2="76.1874" width="0.4064" layer="16"/>
-<wire x1="30.47" y1="76.1874" x2="30.47" y2="80.445" width="0.4064" layer="16"/>
+<wire x1="18.17290625" y1="75.6638" x2="40.588675" y2="75.6638" width="0.4064" layer="1"/>
+<contactref element="U$1" pad="D39"/>
+<wire x1="40.64" y1="75.692" x2="40.64" y2="80.435" width="0.4064" layer="16"/>
+<wire x1="40.64" y1="80.435" x2="40.63" y2="80.445" width="0.4064" layer="16"/>
 </signal>
 <signal name="SDA">
