File: canSim.sch (EAGLE design)
At the start: 16 parts

Commit message: New revision with new OBD-2.  Auto PCB routing to still change.
Parts:
- U$9: value OBD_2FEMALE -> OBD_2FEMALEOBD2_FEMALE_PTH; device OBD2_Female_PTH:OBD_2FEMALE -> OBD2_Female_PTH:OBD_2FEMALEOBD2_FEMALE_PTH
Other:
- moved on the sheet: H1, H2, H3, H4, H5, U$1

Commit message: Release candidate
Parts:
- added R1, R2: 10k, resistor:R-US_0207/2V
- added T1: 2N3904, transistor:2N3904
Connections:
- new net COLL: R2.1, T1.C, U$6.EN
- new net N$2: R1.2, T1.B
- net +5V: now also R2.2
- net 12V_EN: now also R1.1; no longer U$6.EN
- net GND: now also T1.E

Commit message: Swap interrupt and CS pins because some ESP32 pins are input-only.
Connections:
- net CS2: now also U$1.IO32; no longer U$1.VN-IO39
- net CS3: now also U$1.IO33; no longer U$1.IO34
- net INT2_3V3: now also U$1.IO34; no longer U$1.IO32
- net INT3_3V3: now also U$1.VN-IO39; no longer U$1.IO33
Changed lines of the file:
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@@
 <net name="CS2" class="0">
-<segment>
-<pinref part="U$1" gate="G$1" pin="VN-IO39"/>
-<wire x1="93.98" y1="76.2" x2="83.82" y2="76.2" width="0.1524" layer="91"/>
-<label x="83.82" y="76.2" size="1.778" layer="95"/>
-</segment>
 <segment>
 <pinref part="U$3" gate="G$1" pin="CS"/>
@@
 <label x="137.16" y="127" size="1.778" layer="95"/>
 </segment>
+<segment>
+<pinref part="U$1" gate="G$1" pin="IO32"/>
+<wire x1="93.98" y1="68.58" x2="81.28" y2="68.58" width="0.1524" layer="91"/>
+<label x="81.28" y="68.58" size="1.778" layer="95"/>
+</segment>
 </net>
 <net name="CS3" class="0">
-<segment>
-<pinref part="U$1" gate="G$1" pin="IO34"/>
-<wire x1="93.98" y1="73.66" x2="83.82" y2="73.66" width="0.1524" layer="91"/>
-<label x="83.82" y="73.66" size="1.778" layer="95"/>
-</segment>
 <segment>
 <pinref part="U$4" gate="G$1" pin="CS"/>
 <wire x1="165.1" y1="101.6" x2="137.16" y2="101.6" width="0.1524" layer="91"/>
 <label x="137.16" y="101.6" size="1.778" layer="95"/>
+</segment>
+<segment>
+<pinref part="U$1" gate="G$1" pin="IO33"/>
+<wire x1="93.98" y1="66.04" x2="81.28" y2="66.04" width="0.1524" layer="91"/>
+<label x="81.28" y="66.04" size="1.778" layer="95"/>
 </segment>
 </net>
@@
 <net name="INT2_3V3" class="0">
 <segment>
-<pinref part="U$1" gate="G$1" pin="IO32"/>
-<wire x1="73.66" y1="68.58" x2="93.98" y2="68.58" width="0.1524" layer="91"/>
-<label x="73.66" y="68.58" size="1.778" layer="95"/>
-</segment>
-<segment>
 <pinref part="U$5" gate="G$1" pin="LV2"/>
 <wire x1="22.86" y1="127" x2="5.08" y2="127" width="0.1524" layer="91"/>
 <label x="5.08" y="127" size="1.778" layer="95"/>
 </segment>
+<segment>
+<pinref part="U$1" gate="G$1" pin="IO34"/>
+<wire x1="93.98" y1="73.66" x2="73.66" y2="73.66" width="0.1524" layer="91"/>
+<label x="73.66" y="73.66" size="1.778" layer="95"/>
+</segment>
 </net>
 <net name="INT3_3V3" class="0">
-<segment>
-<pinref part="U$1" gate="G$1" pin="IO33"/>
-<wire x1="93.98" y1="66.04" x2="73.66" y2="66.04" width="0.1524" layer="91"/>
-<label x="73.66" y="66.04" size="1.778" layer="95"/>
-</segment>
 <segment>
 <pinref part="U$5" gate="G$1" pin="LV3"/>
@@
 <label x="5.08" y="119.38" size="1.778" layer="95"/>
 </segment>
+<segment>
+<pinref part="U$1" gate="G$1" pin="VN-IO39"/>
+<wire x1="93.98" y1="76.2" x2="73.66" y2="76.2" width="0.1524" layer="91"/>
+<label x="73.66" y="76.2" size="1.778" layer="95"/>
+</segment>
 </net>
